Commit message: fix: 실측 치수 반영 및 체스판 위치 재조정
실측 팔 길이: L1=140mm, L2=155mm, L3=75mm (기존 설계값과 다름)
- utils/ik_solver.py, lagrange.py, sim/env_simple.py L1/L2/L3 수정
- 체스판 위치 재조정: 원점(0.015, -0.115) — 전 칸 도달 가능(최대 263mm < 283mm)
- setup/stl_to_urdf.py 실측 관절 좌표 반영
- test_pipeline.py 테스트 좌표 실측 팔 범위로 수정
- URDF 재생성

테스트: ik ✅ lagrange ✅ full ✅ (토크 전부 한계 이내)

https://claude.ai/code/session_01LH4EnHTZqRnCXBSVhiNqwi

File: setup/urdf/robot_full.urdf (robot description, URDF)
Before this commit: robot chess_arm_full, 4 links, 3 joints
Links:
- link base_link: geometry collision box size=0.0400 0.0400 0.1400; visual box size=0.0400 0.0400 0.1400
- link link1: geometry collision box size=0.0400 0.0400 0.1550; visual box size=0.0400 0.0400 0.1550
- link link2: geometry collision box size=0.0400 0.0400 0.0750; visual box size=0.0400 0.0400 0.0750
Joints:
- joint joint1: origin xyz=0 0 0.2800 rpy=0 0 0 -> xyz=0 0 0.1400 rpy=0 0 0
- joint joint2: origin xyz=0 0 0.2200 rpy=0 0 0 -> xyz=0 0 0.1550 rpy=0 0 0
- joint joint3: origin xyz=0 0 0.0800 rpy=0 0 0 -> xyz=0 0 0.0750 rpy=0 0 0

File: setup/urdf/robot_simple.urdf (robot description, URDF)
Before this commit: robot chess_arm, 4 links, 3 joints
Links:
- link base_link: geometry collision box size=0.0400 0.0400 0.1400; visual box size=0.0400 0.0400 0.1400
- link link1: geometry collision box size=0.0400 0.0400 0.1550; visual box size=0.0400 0.0400 0.1550
- link link2: geometry collision box size=0.0400 0.0400 0.0750; visual box size=0.0400 0.0400 0.0750
Joints:
- joint joint1: origin xyz=0 0 0.2800 rpy=0 0 0 -> xyz=0 0 0.1400 rpy=0 0 0
- joint joint2: origin xyz=0 0 0.2200 rpy=0 0 0 -> xyz=0 0 0.1550 rpy=0 0 0
- joint joint3: origin xyz=0 0 0.0800 rpy=0 0 0 -> xyz=0 0 0.0750 rpy=0 0 0

Commit message: feat: 로봇팔 시각화를 실린더+구 조합으로 개선 (발표/보고서용)
- generate_simple_urdf: 박스 → 실린더(12mm 반지름) + 관절 구(18mm)
- 링크별 색상: base=다크그레이, link1=파랑, link2=초록, end_effector=주황
- 관절 위치를 노란 구로 명시적으로 표시
- robot_simple.urdf, robot_full.urdf 재생성

https://claude.ai/code/session_01LH4EnHTZqRnCXBSVhiNqwi

File: setup/urdf/robot_full.urdf (robot description, URDF)
Before this commit: robot chess_arm_full, 4 links, 3 joints
Links:
- link base_link: mass 0.3 -> 0.12
- link link1: mass 0.2 -> 0.08
- link link2: mass 0.1 -> 0.04
Joints:
- joint joint1: limit lower=-3.14 upper=3.14 effort=1.27 velocity=1.0 -> lower=-3.14 upper=3.14 effort=1.27 velocity=6.0
- joint joint2: limit lower=-1.2 upper=1.2 effort=1.27 velocity=1.0 -> lower=-1.2 upper=1.2 effort=1.27 velocity=6.0
- joint joint3: limit lower=-1.5 upper=1.5 effort=1.27 velocity=1.0 -> lower=-1.5 upper=1.5 effort=1.27 velocity=6.0

File: setup/urdf/robot_simple.urdf (robot description, URDF)
Before this commit: robot chess_arm, 4 links, 3 joints
Links:
- added link base_link_joint_sphere, mass 0.001; visual sphere radius=0.0180
- added link end_effector_joint_sphere, mass 0.001; visual sphere radius=0.0180
- added link link1_joint_sphere, mass 0.001; visual sphere radius=0.0180
- added link link2_joint_sphere, mass 0.001; visual sphere radius=0.0180
- link base_link: mass 0.3 -> 0.12; geometry collision cylinder length=0.1400 radius=0.0120; visual cylinder length=0.1400 radius=0.0120
- link end_effector: mass 0.05 -> 0.03; geometry collision cylinder length=0.0300 radius=0.0120; visual cylinder length=0.0300 radius=0.0120
- link link1: mass 0.2 -> 0.08; geometry collision cylinder length=0.1550 radius=0.0120; visual cylinder length=0.1550 radius=0.0120
- link link2: mass 0.1 -> 0.04; geometry collision cylinder length=0.0750 radius=0.0120; visual cylinder length=0.0750 radius=0.0120
Joints:
- added joint sphere_joint_base_link: type fixed, parent base_link, child base_link_joint_sphere, origin xyz=0 0 0 rpy=0 0 0
- added joint sphere_joint_end_effector: type fixed, parent end_effector, child end_effector_joint_sphere, origin xyz=0 0 0 rpy=0 0 0
- added joint sphere_joint_link1: type fixed, parent link1, child link1_joint_sphere, origin xyz=0 0 0 rpy=0 0 0
- added joint sphere_joint_link2: type fixed, parent link2, child link2_joint_sphere, origin xyz=0 0 0 rpy=0 0 0
- joint joint1: limit lower=-3.14 upper=3.14 effort=1.27 velocity=1.0 -> lower=-3.14 upper=3.14 effort=1.27 velocity=6.0
- joint joint2: limit lower=-1.2 upper=1.2 effort=1.27 velocity=1.0 -> lower=-1.2 upper=1.2 effort=1.27 velocity=6.0
- joint joint3: limit lower=-1.5 upper=1.5 effort=1.27 velocity=1.0 -> lower=-1.5 upper=1.5 effort=1.27 velocity=6.0
